Commit message: Fix base_link URDF mesh reference, add robot model preview and architecture diagrams

File: owr_description/urdf/owr.urdf.xacro (robot description, xacro)
@@ -92,7 +92,4 @@
                     <mesh filename="${bl_stl}" />
                 </geometry>
-                <geometry>
-                    <mesh filename="${bl_dae}"/>
-                </geometry>
                 <material name="LightGrey">
                     <color rgba="0.7 0.7 0.7 1.0"/>
